File: PCB/macropad.kicad_pcb (KiCad board)
At the start: 2 copper layers, 93.5 x 74 mm, 16 parts, among them J1 Conn_01x04, SW1 SW_Push, SW2 SW_Push, SW3 SW_Push, SW4 SW_Push, SW5 SW_Push, SW6 SW_Push, SW7 RotaryEncoder_Switch, U1 MOUDLE-SEEEDUINO-XIAO

Commit message: Add files via upload
Parts:
- J1: footprint Connector_PinHeader_2.54mm:PinHeader_1x04_P2.54mm_Horizontal -> OLED:OLED_0.91_128x32
- moved J1 6.56 mm to (101.0, 109.0), turned to 180 degrees
Routing:
- net VCC: track 64.8 -> 59.8 mm
- net GND: track 94.5 -> 89.6 mm, vias 0 -> 2
- net /EC11A: track 99.3 -> 102.1 mm
- net /SCL: track 43.5 -> 45.1 mm
- net /SDA: track 42.3 -> 41.7 mm, vias 0 -> 2
Other:
- board text added: "Nooruddins BOARD :)"
